Commit message: Edit local planner parameters

File: src/pick_objects/urdf/my_robot.xacro (robot description, xacro)
@@ -79,5 +79,5 @@
   </link>
   <joint type="continuous" name="left_wheel_hinge">
-    <origin xyz="0 0.15 0" rpy="0 0 0"/>
+    <origin xyz="0 0.13 0" rpy="0 0 0"/>
     <child link="left_wheel"/>
     <parent link="chassis"/>
@@ -109,5 +109,5 @@
   </link>
   <joint type="continuous" name="right_wheel_hinge">
-    <origin xyz="0 -0.15 0" rpy="0 0 0"/>
+    <origin xyz="0 -0.13 0" rpy="0 0 0"/>
     <child link="right_wheel"/>
     <parent link="chassis"/>
